File: Electronics/BMS FrontEnd/OpenBMSFrontEnd.kicad_pcb (KiCad board)
At the start: 2 copper layers, 50 x 50 mm, 85 parts, among them J1 CONN_02X05, J2 OpenBMSRiser, J3 VBATT+, J4 VBATT-, J5 PACK+, J6 PACK-, Q1 NDS0605, Q101 FDMS8050, Q102 FDMS8050, Q2 NDS7002A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

Commit message: User Interface board layout rough pass
Other:
- outline, holes or cut-outs redrawn
- net class CellBal: trace_width 0.35 -> 0.2
Changed lines of the file:
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@@
     (area 128.924999 68.924999 179.075001 119.075001)
     (thickness 1.6)
-    (drawings 32)
-    (tracks 665)
+    (drawings 36)
+    (tracks 666)
     (zones 0)
     (modules 85)
@@
     (last_trace_width 0.2)
     (trace_clearance 0.2)
-    (zone_clearance 0.508)
+    (zone_clearance 0.7)
     (zone_45_only no)
     (trace_min 0.2)
@@
   (net_class CellBal ""
     (clearance 0.2)
-    (trace_width 0.35)
+    (trace_width 0.2)
     (via_dia 0.6)
     (via_drill 0.4)
@@
       (net 4 GND))
   )
+  (gr_arc (start 132.5 115.5) (end 132.5 119) (angle 90) (layer Edge.Cuts) (width 0.15))
+  (gr_arc (start 132.5 72.5) (end 129 72.5) (angle 90) (layer Edge.Cuts) (width 0.15))
+  (gr_arc (start 175.5 115.5) (end 179 115.5) (angle 90) (layer Edge.Cuts) (width 0.15))
+  (gr_arc (start 175.5 72.5) (end 175.5 69) (angle 90) (layer Edge.Cuts) (width 0.15))
   (gr_text "OpenBMS\nV2.0" (at 154.1 74.5) (layer B.SilkS)
     (effects (font (size 1.5 1.5) (thickness 0.2)) (justify mirror))
@@
   (gr_line (start 158.4 90.6) (end 158.4 90) (layer F.SilkS) (width 0.2))
   (gr_line (start 158.4 112.6) (end 158.4 90.6) (layer F.SilkS) (width 0.2))
-  (gr_line (start 129 69) (end 179 69) (layer Edge.Cuts) (width 0.15))
-  (gr_line (start 129 119) (end 129 69) (layer Edge.Cuts) (width 0.15))
-  (gr_line (start 179 119) (end 129 119) (layer Edge.Cuts) (width 0.15))
-  (gr_line (start 179 69) (end 179 119) (layer Edge.Cuts) (width 0.15))
+  (gr_line (start 132.5 69) (end 175.5 69) (layer Edge.Cuts) (width 0.15))
+  (gr_line (start 129 115.5) (end 129 72.5) (layer Edge.Cuts) (width 0.15))
+  (gr_line (start 175.5 119) (end 132.5 119) (layer Edge.Cuts) (width 0.15))
+  (gr_line (start 179 72.5) (end 179 115.5) (layer Edge.Cuts) (width 0.15))
   (segment (start 167.85 95.75) (end 167.85 94.818603) (width 0.2) (layer F.Cu) (net 1))
   (segment (start 167.85 94.818603) (end 162.831397 89.8) (width 0.2) (layer F.Cu) (net 1))
@@
   (segment (start 169.45 103.85) (end 170.3 104.7) (width 0.2) (layer F.Cu) (net 3))
   (segment (start 169.45 101.75) (end 169.45 103.85) (width 0.2) (layer F.Cu) (net 3))
+  (segment (start 169.05 101.75) (end 169.05 104.310502) (width 0.2) (layer F.Cu) (net 4))
+  (segment (start 169.05 104.310502) (end 169.138241 104.398743) (width 0.2) (layer F.Cu) (net 4))
+  (via (at 169.138241 104.398743) (size 0.6) (drill 0.4) (layers F.Cu B.Cu) (net 4))
   (segment (start 144.5 111.5) (end 146.3 111.5) (width 0.25) (layer F.Cu) (net 4))
   (segment (start 146.3 111.5) (end 146.5 111.7) (width 0.25) (layer F.Cu) (net 4))
@@
   (segment (start 173.9 99.35) (end 174 99.25) (width 0.2) (layer F.Cu) (net 4))
   (via (at 174 99.25) (size 0.6) (drill 0.4) (layers F.Cu B.Cu) (net 4))
-  (segment (start 169.05 101.75) (end 169.05 104.299417) (width 0.2) (layer F.Cu) (net 4))
-  (segment (start 169.05 104.299417) (end 169.300581 104.549998) (width 0.2) (layer F.Cu) (net 4))
-  (via (at 169.300581 104.549998) (size 0.6) (drill 0.4) (layers F.Cu B.Cu) (net 4))
   (segment (start 171.1 106.95) (end 170.65 106.95) (width 0.2) (layer F.Cu) (net 4))
   (segment (start 170.65 106.95) (end 170.3 107.3) (width 0.2) (layer F.Cu) (net 4))
@@
   (segment (start 161.5 110.25) (end 157.75 110.25) (width 0.2) (layer F.Cu) (net 60))
   (segment (start 168.25 101.75) (end 168.25 103.5) (width 0.2) (layer F.Cu) (net 60))
-  (segment (start 168.65 104.6) (end 161.75 111.5) (width 0.2) (layer F.Cu) (net 61))
-  (segment (start 161.75 111.5) (end 160.75 111.5) (width 0.2) (layer F.Cu) (net 61))
-  (segment (start 168.65 101.75) (end 168.65 104.6) (width 0.2) (layer F.Cu) (net 61))
+  (segment (start 168.65 101.75) (end 168.65 103.3) (width 0.2) (layer F.Cu) (net 61))
+  (segment (start 168.65 104.05) (end 168.65 103.3) (width 0.2) (layer F.Cu) (net 61))
+  (segment (start 160.75 111.5) (end 161.2 111.5) (width 0.2) (layer F.Cu) (net 61))
+  (segment (start 161.2 111.5) (end 168.65 104.05) (width 0.2) (layer F.Cu) (net 61))
   (segment (start 153.4 114) (end 154 114.6) (width 0.2) (layer B.Cu) (net 62))
   (segment (start 154 114.6) (end 154 117) (width 0.2) (layer B.Cu) (net 62))
@@
   (segment (start 170.09 85.6) (end 168.75 84.26) (width 0.2) (layer F.Cu) (net 67))
   (zone (net 4) (net_name GND) (layer B.Cu) (hatch edge 0.508)
-    (connect_pads yes (clearance 0.508))
+    (connect_pads yes (clearance 0.7))
     (min_thickness 0.254)
     (fill yes (arc_segments 16) (thermal_gap 0.508) (thermal_bridge_width 0.508) (smoothing fillet))
